File: dokument/synth_board/synth_board.sch (KiCad schematic (older format))
At the start: 63 parts, among them IC1 ATMEGA1284-P, U1 74LS165, U10 BUTTON, U11 BUTTON, U12 BUTTON, U13 BUTTON, U14 BUTTON, U15 BUTTON, U16 BUTTON, U17 BUTTON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

Commit message: finished with main board, kind of...
Parts:
- added C5, C6: CP1, ~, symbol CP1
- added Q1: BC547, TO92, symbol BC547
- added R33, R34: R, ~, symbol R
- added SP2: SPEAKER, ~, symbol SPEAKER
- added U25: MIC, symbol MIC
- added U26, U?: VCCGND, symbol VCCGND
- added U27: SPANNING_SIGNAL, symbol SPANNING_SIGNAL
Connections:
- net at IC1.31 (GND), ISP1.6 (GND), R21.2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: now also U27.3 (GND), U?.2 (GND)
- net at IC1.29 ((PCINT23/TOSC2)PC7), R8.1: now also U27.2 (SIGNAL)
- net at IC1.10 (VCC), ISP1.2 (VCC), U1.16 (VCC)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: now also U27.1 (VCC), U?.1 (VCC)
- new net: C5.2, U25.1 (ELEC+)
- new net: Q1.3 (E), SP2.2, U25.2 (GND), U26.2 (GND)
- new net: C6.1, Q1.1 (C), R33.2, R34.2
- new net: C5.1, Q1.2 (B), R33.1
- new net: C6.2, SP2.1
- new net: R34.1, U26.1 (VCC)
Changed lines of the file:
@@
 	2650 3650 2800 3650
 Wire Wire Line
-	2800 3650 2800 5550
+	2800 3650 2800 5650
 Wire Wire Line
 	2800 5550 3200 5550
 Wire Wire Line
-	1650 5800 4950 5800
+	1650 5800 5100 5800
 Wire Wire Line
 	4950 550  4950 800
@@
 Connection ~ 1650 5050
 Wire Wire Line
-	1800 5150 700  5150
+	550  5150 1800 5150
 Wire Wire Line
 	700  5150 700  2500
@@
 	8450 4450 8750 4450
 Wire Wire Line
-	8750 4450 8750 6000
-Wire Wire Line
-	8750 6000 6750 6000
-Wire Wire Line
-	6750 6000 6750 5800
-Wire Wire Line
 	4250 6100 4250 6300
 Wire Wire Line
@@
 Wire Wire Line
 	1800 5250 1750 5250
+$Comp
+L MIC U25
+U 1 1 544CF6E6
+P 8000 6550
+F 0 "U25" H 8000 6400 60  0000 C CNN
+F 1 "MIC" H 8000 6700 60  0000 C CNN
+F 2 "" H 8000 6550 60  0000 C CNN
+F 3 "" H 8000 6550 60  0000 C CNN
+	1    8000 6550
+	0    1    1    0
+$EndComp
+Wire Wire Line
+	6750 5550 8750 5550
+Wire Wire Line
+	6750 5800 6750 5550
+Wire Wire Line
+	8750 5550 8750 4450
+$Comp
+L BC547 Q1
+U 1 1 544CFD93
+P 9150 6750
+F 0 "Q1" H 9150 6601 40  0000 R CNN
+F 1 "BC547" H 9150 6900 40  0000 R CNN
+F 2 "TO92" H 9050 6852 29  0000 C CNN
+F 3 "~" H 9150 6750 60  0000 C CNN
+	1    9150 6750
+	1    0    0    -1
+$EndComp
+$Comp
+L CP1 C6
+U 1 1 544CFEEA
+P 9550 6350
+F 0 "C6" H 9600 6450 50  0000 L CNN
+F 1 "CP1" H 9600 6250 50  0000 L CNN
+F 2 "~" H 9550 6350 60  0000 C CNN
+F 3 "~" H 9550 6350 60  0000 C CNN
+	1    9550 6350
+	0    -1   -1   0
+$EndComp
+$Comp
+L CP1 C5
+U 1 1 544CFEF9
+P 8550 6500
+F 0 "C5" H 8600 6600 50  0000 L CNN
+F 1 "CP1" H 8600 6400 50  0000 L CNN
+F 2 "~" H 8550 6500 60  0000 C CNN
+F 3 "~" H 8550 6500 60  0000 C CNN
+	1    8550 6500
+	0    1    1    0
+$EndComp
+$Comp
+L R R33
+U 1 1 544D283E
+P 9000 6350
+F 0 "R33" V 9080 6350 40  0000 C CNN
+F 1 "R" V 9007 6351 40  0000 C CNN
+F 2 "~" V 8930 6350 30  0000 C CNN
+F 3 "~" H 9000 6350 30  0000 C CNN
+	1    9000 6350
+	0    -1   -1   0
+$EndComp
+$Comp
+L R R34
+U 1 1 544D284D
+P 9250 6050
+F 0 "R34" V 9330 6050 40  0000 C CNN
+F 1 "R" V 9257 6051 40  0000 C CNN
+F 2 "~" V 9180 6050 30  0000 C CNN
+F 3 "~" H 9250 6050 30  0000 C CNN
+	1    9250 6050
+	1    0    0    -1
+$EndComp
+Wire Wire Line
+	8000 5950 8350 5950
+Wire Wire Line
+	8350 5950 8350 6500
+Wire Wire Line
+	8750 6350 8750 6750
+Wire Wire Line
+	9250 6300 9250 6550
+Wire Wire Line
+	9350 6350 9250 6350
+Wire Wire Line
+	9250 6950 9250 7100
+Wire Wire Line
+	8000 7100 11050 7100
+Connection ~ 9250 6350
+Wire Wire Line
+	8750 6750 8950 6750
+Connection ~ 8750 6500
+$Comp
+L VCCGND U26
+U 1 1 544D426E
+P 10550 6350
+F 0 "U26" H 10550 6150 60  0000 C CNN
+F 1 "VCCGND" H 10550 6500 60  0000 C CNN
+F 2 "" H 10550 6350 60  0000 C CNN
+F 3 "" H 10550 6350 60  0000 C CNN
+	1    10550 6350
+	1    0    0    -1
+$EndComp
+Wire Wire Line
+	9250 5800 9600 5800
+Wire Wire Line
+	9600 5800 9600 6050
+Wire Wire Line
+	9600 6050 10050 6050
+Wire Wire Line
+	10050 6050 10050 6350
+Wire Wire Line
+	11050 7100 11050 6350
+Connection ~ 9250 7100
+$Comp
+L SPEAKER SP2
+U 1 1 544D455C
+P 10050 6750
+F 0 "SP2" H 9950 7000 70  0000 C CNN
+F 1 "SPEAKER" H 9950 6500 70  0000 C CNN
+F 2 "~" H 10050 6750 60  0000 C CNN
+F 3 "~" H 10050 6750 60  0000 C CNN
+	1    10050 6750
+	1    0    0    -1
+$EndComp
+Wire Wire Line
+	9750 6350 9750 6650
+Wire Wire Line
+	9750 6850 9750 7100
+Connection ~ 9750 7100
+$Comp
+L SPANNING_SIGNAL U27
+U 1 1 544D49D4
+P 4550 4750
+F 0 "U27" H 4550 4550 60  0000 C CNN
+F 1 "SPANNING_SIGNAL" H 4550 4950 60  0000 C CNN
+F 2 "" H 4550 4850 60  0000 C CNN
+F 3 "" H 4550 4850 60  0000 C CNN
+	1    4550 4750
+	1    0    0    -1
+$EndComp
+Wire Wire Line
+	5100 5800 5100 4750
+Connection ~ 4950 5800
+Wire Wire Line
+	2800 5650 4550 5650
+Wire Wire Line
+	4550 5650 4550 5200
+Connection ~ 2800 5550
+Wire Wire Line
+	4000 1350 4000 4750
+Wire Wire Line
+	4000 1350 3450 1350
+Wire Wire Line
+	3450 1350 3450 550
+Connection ~ 3450 550
+$Comp
+L VCCGND U?
+U 1 1 544D4FEF
+P 1050 5450
+F 0 "U?" H 1050 5250 60  0000 C CNN
+F 1 "VCCGND" H 1050 5600 60  0000 C CNN
+F 2 "" H 1050 5450 60  0000 C CNN
+F 3 "" H 1050 5450 60  0000 C CNN
+	1    1050 5450
+	1    0    0    -1
+$EndComp
+Wire Wire Line
+	1550 5450 1650 5450
+Connection ~ 1650 5450
+Wire Wire Line
+	550  5450 550  5150
+Connection ~ 700  5150
 $EndSCHEMATC

Commit message: just going to add pot and electret mic
Parts:
- added C7: C, ~, symbol C
- added RV?: POT, ~, symbol POT
- added U29: 4BUTTON, symbol 4BUTTON
- added U?: MIC, symbol MIC
- added X1: CRYSTAL, ~, symbol CRYSTAL
- gave numbers to parts that had none: 1
Connections:
- net at IC1.31 (GND), ISP1.6 (GND), R21.2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: now also C7.2, RV?.1
- net at IC1.1 ((PCINT8/T0/XCK)PB0), U1.1 (Pl): now also U2.1 (Pl)
- net at IC1.10 (VCC), ISP1.2 (VCC), U1.16 (VCC)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: now also IC1.30 (AVCC), RV?.3, U29.5 (VCC)
- net at IC1.12 (XTAL2): now also X1.2
- net at IC1.13 (XTAL1): now also X1.1
- net at IC1.2 ((PCINT9/CLKO/T1)PB1): now also U29.2
- net at IC1.20 ((PCINT30/OC2B/ICP)PD6): now also U29.1
- net at IC1.3 ((PCINT10/AIN0/INT2)PB2): now also U29.3
- net at IC1.32 (AREF): now also C7.1
- net at IC1.4 ((PCINT11/AIN1/OC0)PB3): now also U29.4
- net at IC1.40 ((PCINT0/ADC0)PA0): now also RV?.2
- net at IC1.7 ((PCINT14/MISO)PB6), ISP1.1 (MISO): now also U2.9 (Q7)
Changed lines of the file:
@@
 	1    0    0    -1
 $EndComp
+$Comp
+L MIC U25
+U 1 1 544CF6E6
+P 8000 6550
+F 0 "U25" H 8000 6400 60  0000 C CNN
+F 1 "MIC" H 8000 6700 60  0000 C CNN
+F 2 "" H 8000 6550 60  0000 C CNN
+F 3 "" H 8000 6550 60  0000 C CNN
+	1    8000 6550
+	0    1    1    0
+$EndComp
+$Comp
+L BC547 Q1
+U 1 1 544CFD93
+P 9150 6750
+F 0 "Q1" H 9150 6601 40  0000 R CNN
+F 1 "BC547" H 9150 6900 40  0000 R CNN
+F 2 "TO92" H 9050 6852 29  0000 C CNN
+F 3 "~" H 9150 6750 60  0000 C CNN
+	1    9150 6750
+	1    0    0    -1
+$EndComp
+$Comp
+L CP1 C6
+U 1 1 544CFEEA
+P 9550 6350
+F 0 "C6" H 9600 6450 50  0000 L CNN
+F 1 "CP1" H 9600 6250 50  0000 L CNN
+F 2 "~" H 9550 6350 60  0000 C CNN
+F 3 "~" H 9550 6350 60  0000 C CNN
+	1    9550 6350
+	0    -1   -1   0
+$EndComp
+$Comp
+L CP1 C5
+U 1 1 544CFEF9
+P 8550 6500
+F 0 "C5" H 8600 6600 50  0000 L CNN
+F 1 "CP1" H 8600 6400 50  0000 L CNN
+F 2 "~" H 8550 6500 60  0000 C CNN
+F 3 "~" H 8550 6500 60  0000 C CNN
+	1    8550 6500
+	0    1    1    0
+$EndComp
+$Comp
+L R R33
+U 1 1 544D283E
+P 9000 6350
+F 0 "R33" V 9080 6350 40  0000 C CNN
+F 1 "R" V 9007 6351 40  0000 C CNN
+F 2 "~" V 8930 6350 30  0000 C CNN
+F 3 "~" H 9000 6350 30  0000 C CNN
+	1    9000 6350
+	0    -1   -1   0
+$EndComp
+$Comp
+L R R34
+U 1 1 544D284D
+P 9250 6050
+F 0 "R34" V 9330 6050 40  0000 C CNN
+F 1 "R" V 9257 6051 40  0000 C CNN
+F 2 "~" V 9180 6050 30  0000 C CNN
+F 3 "~" H 9250 6050 30  0000 C CNN
+	1    9250 6050
+	1    0    0    -1
+$EndComp
+$Comp
+L VCCGND U26
+U 1 1 544D426E
+P 10550 6350
+F 0 "U26" H 10550 6150 60  0000 C CNN
+F 1 "VCCGND" H 10550 6500 60  0000 C CNN
+F 2 "" H 10550 6350 60  0000 C CNN
+F 3 "" H 10550 6350 60  0000 C CNN
+	1    10550 6350
+	1    0    0    -1
+$EndComp
+$Comp
+L SPEAKER SP2
+U 1 1 544D455C
+P 10050 6750
+F 0 "SP2" H 9950 7000 70  0000 C CNN
+F 1 "SPEAKER" H 9950 6500 70  0000 C CNN
+F 2 "~" H 10050 6750 60  0000 C CNN
+F 3 "~" H 10050 6750 60  0000 C CNN
+	1    10050 6750
+	1    0    0    -1
+$EndComp
+$Comp
+L SPANNING_SIGNAL U27
+U 1 1 544D49D4
+P 4550 4750
+F 0 "U27" H 4550 4550 60  0000 C CNN
+F 1 "SPANNING_SIGNAL" H 4550 4950 60  0000 C CNN
+F 2 "" H 4550 4850 60  0000 C CNN
+F 3 "" H 4550 4850 60  0000 C CNN
+	1    4550 4750
+	1    0    0    -1
+$EndComp
+$Comp
+L VCCGND U28
+U 1 1 544D4FEF
+P 1050 5450
+F 0 "U28" H 1050 5250 60  0000 C CNN
+F 1 "VCCGND" H 1050 5600 60  0000 C CNN
+F 2 "" H 1050 5450 60  0000 C CNN
+F 3 "" H 1050 5450 60  0000 C CNN
+	1    1050 5450
+	1    0    0    -1
+$EndComp
+$Comp
+L C C7
+U 1 1 544D6FCC
+P 650 2550
+F 0 "C7" H 650 2650 40  0000 L CNN
+F 1 "C" H 656 2465 40  0000 L CNN
+F 2 "~" H 688 2400 30  0000 C CNN
+F 3 "~" H 650 2550 60  0000 C CNN
+	1    650  2550
+	1    0    0    -1
+$EndComp
+$Comp
+L 4BUTTON U29
+U 1 1 544D72E5
+P 1250 6150
+F 0 "U29" H 1250 5950 60  0000 C CNN
+F 1 "4BUTTON" H 1250 6350 60  0000 C CNN
+F 2 "" H 1250 6150 60  0000 C CNN
+F 3 "" H 1250 6150 60  0000 C CNN
+	1    1250 6150
+	1    0    0    -1
+$EndComp
 Wire Wire Line
 	2650 2950 3050 2950
@@
 	4750 2650 5150 2650
 Wire Wire Line
-	1800 5050 1650 5050
+	600  5050 1800 5050
 Connection ~ 1650 5050
 Wire Wire Line
@@
 	3000 2400 4800 2400
 Wire Wire Line
-	4800 2400 4800 2500
+	4800 2400 4800 2850
 Wire Wire Line
 	4800 2500 5150 2500
@@
 Connection ~ 5800 800
 Wire Wire Line
-	4950 2400 6000 2400
+	4850 2400 6000 2400
 Connection ~ 6000 2400
 Connection ~ 4950 2400
@@
 Wire Wire Line
 	1800 5250 1750 5250
-$Comp
-L MIC U25
-U 1 1 544CF6E6
-P 8000 6550
-F 0 "U25" H 8000 6400 60  0000 C CNN
-F 1 "MIC" H 8000 6700 60  0000 C CNN
-F 2 "" H 8000 6550 60  0000 C CNN
-F 3 "" H 8000 6550 60  0000 C CNN
-	1    8000 6550
-	0    1    1    0
-$EndComp
 Wire Wire Line
 	6750 5550 8750 5550
@@
 Wire Wire Line
 	8750 5550 8750 4450
-$Comp
-L BC547 Q1
-U 1 1 544CFD93
-P 9150 6750
-F 0 "Q1" H 9150 6601 40  0000 R CNN
-F 1 "BC547" H 9150 6900 40  0000 R CNN
-F 2 "TO92" H 9050 6852 29  0000 C CNN
-F 3 "~" H 9150 6750 60  0000 C CNN
-	1    9150 6750
-	1    0    0    -1
-$EndComp
-$Comp
-L CP1 C6
-U 1 1 544CFEEA
-P 9550 6350
-F 0 "C6" H 9600 6450 50  0000 L CNN
-F 1 "CP1" H 9600 6250 50  0000 L CNN
-F 2 "~" H 9550 6350 60  0000 C CNN
-F 3 "~" H 9550 6350 60  0000 C CNN
-	1    9550 6350
-	0    -1   -1   0
-$EndComp
-$Comp
-L CP1 C5
-U 1 1 544CFEF9
-P 8550 6500
-F 0 "C5" H 8600 6600 50  0000 L CNN
-F 1 "CP1" H 8600 6400 50  0000 L CNN
-F 2 "~" H 8550 6500 60  0000 C CNN
-F 3 "~" H 8550 6500 60  0000 C CNN
-	1    8550 6500
-	0    1    1    0
-$EndComp
-$Comp
-L R R33
-U 1 1 544D283E
-P 9000 6350
-F 0 "R33" V 9080 6350 40  0000 C CNN
-F 1 "R" V 9007 6351 40  0000 C CNN
-F 2 "~" V 8930 6350 30  0000 C CNN
-F 3 "~" H 9000 6350 30  0000 C CNN
-	1    9000 6350
-	0    -1   -1   0
-$EndComp
-$Comp
-L R R34
-U 1 1 544D284D
-P 9250 6050
-F 0 "R34" V 9330 6050 40  0000 C CNN
-F 1 "R" V 9257 6051 40  0000 C CNN
-F 2 "~" V 9180 6050 30  0000 C CNN
-F 3 "~" H 9250 6050 30  0000 C CNN
-	1    9250 6050
-	1    0    0    -1
-$EndComp
 Wire Wire Line
 	8000 5950 8350 5950
@@
 	8750 6750 8950 6750
 Connection ~ 8750 6500
-$Comp
-L VCCGND U26
-U 1 1 544D426E
-P 10550 6350
-F 0 "U26" H 10550 6150 60  0000 C CNN
-F 1 "VCCGND" H 10550 6500 60  0000 C CNN
-F 2 "" H 10550 6350 60  0000 C CNN
-F 3 "" H 10550 6350 60  0000 C CNN
-	1    10550 6350
-	1    0    0    -1
-$EndComp
 Wire Wire Line
 	9250 5800 9600 5800
@@
 	11050 7100 11050 6350
 Connection ~ 9250 7100
-$Comp
-L SPEAKER SP2
-U 1 1 544D455C
-P 10050 6750
-F 0 "SP2" H 9950 7000 70  0000 C CNN
-F 1 "SPEAKER" H 9950 6500 70  0000 C CNN
-F 2 "~" H 10050 6750 60  0000 C CNN
-F 3 "~" H 10050 6750 60  0000 C CNN
-	1    10050 6750
-	1    0    0    -1
-$EndComp
 Wire Wire Line
 	9750 6350 9750 6650
@@
 	9750 6850 9750 7100
 Connection ~ 9750 7100
-$Comp
-L SPANNING_SIGNAL U27
-U 1 1 544D49D4
-P 4550 4750
-F 0 "U27" H 4550 4550 60  0000 C CNN
-F 1 "SPANNING_SIGNAL" H 4550 4950 60  0000 C CNN
-F 2 "" H 4550 4850 60  0000 C CNN
-F 3 "" H 4550 4850 60  0000 C CNN
-	1    4550 4750
-	1    0    0    -1
-$EndComp
 Wire Wire Line
 	5100 5800 5100 4750
@@
 	4000 1350 4000 4750
 Wire Wire Line
-	4000 1350 3450 1350
+	3250 1350 4000 1350
 Wire Wire Line
 	3450 1350 3450 550
 Connection ~ 3450 550
-$Comp
-L VCCGND U?
-U 1 1 544D4FEF
-P 1050 5450
-F 0 "U?" H 1050 5250 60  0000 C CNN
-F 1 "VCCGND" H 1050 5600 60  0000 C CNN
-F 2 "" H 1050 5450 60  0000 C CNN
-F 3 "" H 1050 5450 60  0000 C CNN
-	1    1050 5450
-	1    0    0    -1
-$EndComp
 Wire Wire Line
 	1550 5450 1650 5450
 Connection ~ 1650 5450
 Wire Wire Line
-	550  5450 550  5150
+	550  5150 550  6450
 Connection ~ 700  5150
+Wire Wire Line
+	4800 2850 4300 2850
+Wire Wire Line
+	4300 2850 4300 3950
+Wire Wire Line
+	4300 3950 5150 3950
+Connection ~ 4800 2500
+Wire Wire Line
+	3650 800  3650 650
+Wire Wire Line
+	3650 650  6750 650
+Wire Wire Line
+	6750 650  6750 3100
+Wire Wire Line
+	6750 3100 6550 3100
+Connection ~ 3650 800
+Wire Wire Line
+	1450 850  1650 850
+Wire Wire Line
+	600  5050 600  2750
+Wire Wire Line
+	600  2750 650  2750
+Wire Wire Line
+	550  6450 1700 6450
+Wire Wire Line
+	1700 6450 1700 6250
+Connection ~ 550  5450
+Wire Wire Line
+	2650 4450 2850 4450
+Wire Wire Line
+	2850 4450 2850 5850
+Wire Wire Line
+	2850 5850 800  5850
+Wire Wire Line
+	800  5850 800  6050
+$Comp
+L CRYSTAL X1
+U 1 1 544D7B55
+P 1150 1750
+F 0 "X1" H 1150 1900 60  0000 C CNN
+F 1 "CRYSTAL" H 1150 1600 60  0000 C CNN
+F 2 "~" H 1150 1750 60  0000 C CNN
+F 3 "~" H 1150 1750 60  0000 C CNN
+	1    1150 1750
+	0    -1   -1   0
+$EndComp
+Wire Wire Line
+	650  1550 650  1450
+Wire Wire Line
+	650  1450 1150 1450
+Wire Wire Line
+	1150 2050 650  2050
+Wire Wire Line
+	650  2050 650  1950
+Wire Wire Line
+	2650 2150 1100 2150
+Wire Wire Line
+	1100 2150 1100 4950
+Wire Wire Line
+	1100 4950 500  4950
+Wire Wire Line
+	500  4950 500  6150
+Wire Wire Line
+	500  6150 800  6150
+Wire Wire Line
+	2650 2250 1200 2250
+Wire Wire Line
+	1200 2250 1200 4950
+Wire Wire Line
+	1200 4950 1300 4950
+Wire Wire Line
+	1300 4950 1300 5750
+Wire Wire Line
+	1300 5750 1550 5750
+Wire Wire Line
+	1550 5750 1550 5950
+Wire Wire Line
+	1550 5950 1700 5950
+Wire Wire Line
+	1700 5950 1700 6050
+Wire Wire Line
+	2650 2350 1300 2350
+Wire Wire Line
+	1300 2350 1300 4850
+Wire Wire Line
+	1300 4850 1350 4850
+Wire Wire Line
+	1350 4850 1350 5650
+Wire Wire Line
+	1350 5650 1600 5650
+Wire Wire Line
+	1600 5650 1600 5900
+Wire Wire Line
+	1600 5900 1800 5900
+Wire Wire Line
+	1800 5900 1800 6150
+Wire Wire Line
+	1800 6150 1700 6150
+$Comp
+L POT RV?
+U 1 1 544D86AD
+P 3250 1750
+F 0 "RV?" H 3250 1650 50  0000 C CNN
+F 1 "POT" H 3250 1750 50  0000 C CNN
+F 2 "~" H 3250 1750 60  0000 C CNN
+F 3 "~" H 3250 1750 60  0000 C CNN
+	1    3250 1750
+	0    -1   -1   0
+$EndComp
+Wire Wire Line
+	3250 2000 3250 2350
+Wire Wire Line
+	3250 2350 4850 2350
+Wire Wire Line
+	4850 2350 4850 2400
+Wire Wire Line
+	3250 1500 3250 1350
+Connection ~ 3450 1350
+Wire Wire Line
+	2650 1150 3050 1150
+Wire Wire Line
+	3050 1150 3050 1750
+Wire Wire Line
+	3050 1750 3100 1750
+$Comp
+L MIC U?
+U 1 1 544D8E5D
+P 5900 5800
+F 0 "U?" H 5900 5650 60  0000 C CNN
+F 1 "MIC" H 5900 5950 60  0000 C CNN
+F 2 "" H 5900 5800 60  0000 C CNN
+F 3 "" H 5900 5800 60  0000 C CNN
+	1    5900 5800
+	1    0    0    -1
+$EndComp
 $EndSCHEMATC

Commit message: finished yeeeey
Parts:
- removed U?: MIC, symbol MIC
- added U30: VCCGND, symbol VCCGND
- added U31: MIC_INPUT, symbol MIC_INPUT
- gave numbers to parts that had none: 1
Connections:
- net at C7.2, IC1.31 (GND), ISP1.6 (GND)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: now also U30.2 (GND)
- net at IC1.10 (VCC), IC1.30 (AVCC), ISP1.2 (VCC)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: now also U30.1 (VCC)
- net at IC1.33 ((PCINT7/ADC7)PA7): now also U31.1 (input)
Changed lines of the file:
@@
 Connection ~ 1650 5450
 Wire Wire Line
-	550  5150 550  6450
+	550  5150 550  6750
 Connection ~ 700  5150
 Wire Wire Line
@@
 	1800 6150 1700 6150
 $Comp
-L POT RV?
+L POT RV1
 U 1 1 544D86AD
 P 3250 1750
-F 0 "RV?" H 3250 1650 50  0000 C CNN
+F 0 "RV1" H 3250 1650 50  0000 C CNN
 F 1 "POT" H 3250 1750 50  0000 C CNN
 F 2 "~" H 3250 1750 60  0000 C CNN
@@
 	3050 1750 3100 1750
 $Comp
-L MIC U?
-U 1 1 544D8E5D
-P 5900 5800
-F 0 "U?" H 5900 5650 60  0000 C CNN
-F 1 "MIC" H 5900 5950 60  0000 C CNN
-F 2 "" H 5900 5800 60  0000 C CNN
-F 3 "" H 5900 5800 60  0000 C CNN
-	1    5900 5800
+L VCCGND U30
+U 1 1 544D8FB0
+P 1050 6750
+F 0 "U30" H 1050 6550 60  0000 C CNN
+F 1 "VCCGND" H 1050 6900 60  0000 C CNN
+F 2 "" H 1050 6750 60  0000 C CNN
+F 3 "" H 1050 6750 60  0000 C CNN
+	1    1050 6750
 	1    0    0    -1
 $EndComp
+Connection ~ 550  6450
+Wire Wire Line
+	1550 6750 1550 7100
+Wire Wire Line
+	1550 7100 700  7100
+Wire Wire Line
+	700  7100 700  5700
+Wire Wire Line
+	700  5700 1650 5700
+Connection ~ 1650 5700
+$Comp
+L MIC_INPUT U31
+U 1 1 544D9C93
+P 1400 1350
+F 0 "U31" H 1400 1250 60  0000 C CNN
+F 1 "MIC_INPUT" H 1400 1450 60  0000 C CNN
+F 2 "" H 1400 1350 60  0000 C CNN
+F 3 "" H 1400 1350 60  0000 C CNN
+	1    1400 1350
+	-1   0    0    1
+$EndComp
+Wire Wire Line
+	1850 1350 1850 1900
+Wire Wire Line
+	1850 1900 2650 1900
+Wire Wire Line
+	2650 1900 2650 1850
 $EndSCHEMATC
